File: TPS54331_BuckConverter/TPS54331_BuckConverter.kicad_sch (KiCad schematic)
At the start: 0 parts

Commit message: improved schematic photo
Parts:
- added C1, C2: 4.7uF, Capacitor_SMD:C_0805_2012Metric, symbol Device:C
- added C3, C5: 0.01uF, Capacitor_SMD:C_0603_1608Metric, symbol Device:C
- added C4: 0.1uF, Capacitor_SMD:C_0603_1608Metric, symbol Device:C
- added C6: 1000pF, Capacitor_SMD:C_0603_1608Metric, symbol Device:C
- added C7: 47pF, Capacitor_SMD:C_0603_1608Metric, symbol Device:C
- added C8, C9: 47uF, Capacitor_SMD:C_1206_3216Metric, symbol Device:C
- added D1: MB340A, Diode_SMD:D_SMA, symbol Device:D
- added J1, J2, J3, J4: Conn_01x02_Pin, Connector_PinHeader_2.54mm:PinHeader_1x02_P2.54mm_Vertical, symbol Connector:Conn_01x02_Pin
- added L1: 6.8uH, Inductor_SMD:L_10.4x10.4_H4.8, symbol Device:L
- added R1: 332k, Resistor_SMD:R_0603_1608Metric, symbol Device:R
- added R2: 68.1k, Resistor_SMD:R_0603_1608Metric, symbol Device:R
- added R3: 29.4k, Resistor_SMD:R_0603_1608Metric, symbol Device:R
- added R4: 0, Resistor_SMD:R_0603_1608Metric, symbol Device:R
- added R5: 10.2k, Resistor_SMD:R_0603_1608Metric, symbol Device:R
- added R6: 1.96k, Resistor_SMD:R_0603_1608Metric, symbol Device:R
- added TP1, TP2, TP3, TP4, TP5, TP6: TestPoint, TestPoint:TestPoint_Pad_D1.0mm, symbol Connector:TestPoint
- added U1: TPS54331D, Package_SO:SOIC-8_3.9x4.9mm_P1.27mm, symbol Regulator_Switching:TPS54331D
Connections:
- new net: C6.1, C7.1, U1.6 (COMP)
- new net: C6.2, R3.1
- new net: C4.2, D1.1 (K), L1.1, TP3.1, U1.8 (PH)
- new net: R4.2, R5.1, TP4.1
- new net: R5.2, R6.1, U1.5 (VSNS)
- new net: C4.1, U1.1 (BOOT)
- new net EN: J2.1 (Pin_1), R1.2, R2.1, U1.3 (EN)
- new net GND: C1.2, C2.2, C3.2, C5.1, C7.2, C8.2, C9.2, D1.2 (A), J1.1 (Pin_1), J2.2 (Pin_2), J3.2 (Pin_2), J4.2 (Pin_2), R2.2, R3.2, R6.2, TP2.1, TP6.1, U1.7 (GND)
- new net TR: C5.2, J3.1 (Pin_1), U1.4 (SS)
- new net VIN: C1.1, C2.1, C3.1, J1.2 (Pin_2), R1.1, TP1.1, U1.2 (VIN)
- new net VOUT: C8.1, C9.1, J4.1 (Pin_1), L1.2, R4.1, TP5.1
Other:
- title: (none) -> TPS54331_BuckConverter
